Commit message: applying a 3rd approach

File: src/environment/urdf/obj.urdf (robot description, URDF)
Before this commit: robot my_object, 1 links, 0 joints
Links:
- link object_link: geometry collision mesh filename=package://environment/meshes/obj.stl scale=3 3 3; visual mesh filename=package://environment/meshes/obj.stl scale=3 3 3

Commit message: corrected  ap5 best so far

File: src/environment/urdf/obj.urdf (robot description, URDF)
Before this commit: robot my_object, 1 links, 0 joints
Links:
- link object_link: geometry collision mesh filename=package://environment/meshes/obj.stl scale=2.2 2.2 2.2; visual mesh filename=package://environment/meshes/obj.stl scale=2.2 2.2 2.2
